File: pcb/Powersupply-lower.kicad_sch (KiCad schematic)
At the start: 21 parts, among them U3 TPS54294PWP

Commit message: pcb: connect upper and lower
Connections:
- net out_left renamed lower_left
- net out_right renamed lower_right
Changed lines of the file:
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@@
 		)
 	)
-	(hierarchical_label "out_left"
+	(hierarchical_label "lower_left"
 		(shape bidirectional)
 		(at 62.23 38.1 0)
@@
 		)
 	)
-	(hierarchical_label "out_right"
+	(hierarchical_label "lower_right"
 		(shape bidirectional)
 		(at 200.66 27.94 0)
