File: pcb/Powersupply-upper.kicad_sch (KiCad schematic)
At the start: 1 part, among them U2 TPS54325PWP

Commit message: pcp setup
Parts:
- removed U2: TPS54325PWP, PWP14_2P31X2P46, symbol TPS54325:TPS54325PWP
- added U1: TPS54325PWP.d, PWP14_2P31X2P46, symbol TPS54325:TPS54325PWP.d
Other:
- removed sheet Powersupply
Changed lines of the file:
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@@
 	(paper "A4")
 	(symbol
-		(lib_id "TPS54325:TPS54325PWP")
-		(at 193.04 67.31 0)
+		(lib_id "TPS54325:TPS54325PWP.d")
+		(at 59.69 22.86 0)
 		(unit 1)
 		(body_style 1)
@@
 		(dnp no)
 		(fields_autoplaced yes)
-		(property "Reference" "U2"
-			(at 240.03 74.93 0)
+		(property "Reference" "U1"
+			(at 116.84 30.48 0)
 			(show_name no)
 			(do_not_autoplace no)
@@
 			)
 		)
-		(property "Value" "TPS54325PWP"
-			(at 240.03 77.47 0)
+		(property "Value" "TPS54325PWP.d"
+			(at 116.84 33.02 0)
 			(show_name no)
 			(do_not_autoplace no)
@@
 		)
 		(property "Footprint" "PWP14_2P31X2P46"
-			(at 207.01 85.09 0)
+			(at 68.58 67.31 0)
 			(hide yes)
 			(show_name no)
@@
 		)
 		(property "Datasheet" "https://www.ti.com/lit/gpn/tps54325"
-			(at 193.04 67.31 0)
+			(at 59.69 22.86 0)
 			(hide yes)
 			(show_name no)
@@
 		)
 		(property "Description" ""
-			(at 193.04 67.31 0)
+			(at 59.69 22.86 0)
 			(hide yes)
 			(show_name no)
@@
 			)
 		)
-		(pin "9"
+		(pin "3"
 		)
-		(pin "3"
+		(pin "4"
 		)
 		(pin "5"
 		)
-		(pin "4"
+		(pin "6"
+		)
+		(pin "7"
+		)
+		(pin "8"
+		)
+		(pin "12"
+		)
+		(pin "13"
+		)
+		(pin "11"
+		)
+		(pin "2"
+		)
+		(pin "1"
+		)
+		(pin "15"
+		)
+		(pin "9"
+		)
+		(pin "10"
 		)
 		(pin "14"
 		)
-		(pin "10"
-		)
-		(pin "15"
-		)
-		(pin "12"
-		)
-		(pin "6"
-		)
-		(pin "13"
-		)
-		(pin "8"
-		)
-		(pin "1"
-		)
-		(pin "2"
-		)
-		(pin "11"
-		)
-		(pin "7"
-		)
 		(instances
 			(project "tdt4295"
-				(path "/603dd496-f9c4-4a31-9104-19eec41ebc98"
-					(reference "U2")
+				(path "/603dd496-f9c4-4a31-9104-19eec41ebc98/634870db-7705-458e-b29f-8b3e7772e7aa/29fcc9f6-3628-4988-aed7-ebf94d0e9351"
+					(reference "U1")
 					(unit 1)
 				)
@@
 		)
 	)
-	(sheet
-		(at 25.4 38.1)
-		(size 25.4 12.7)
-		(exclude_from_sim no)
-		(in_bom yes)
-		(on_board yes)
-		(dnp no)
-		(fields_autoplaced yes)
-		(stroke
-			(width 0.1524)
-			(type solid)
-		)
-		(fill
-			(color 0 0 0 0)
-		)
-		(property "Sheetname" "Powersupply"
-			(at 25.4 37.3884 0)
-			(show_name no)
-			(do_not_autoplace no)
-			(effects
-				(font
-					(size 1.27 1.27)
-				)
-				(justify left bottom)
-			)
-		)
-		(property "Sheetfile" "Powersupply.kicad_sch"
-			(at 25.4 51.3846 0)
-			(show_name no)
-			(do_not_autoplace no)
-			(effects
-				(font
-					(size 1.27 1.27)
-				)
-				(justify left top)
-			)
-		)
-		(instances
-			(project "tdt4295"
-				(path "/603dd496-f9c4-4a31-9104-19eec41ebc98"
-					(page "4")
-				)
-			)
-		)
-	)
-	(sheet_instances
-		(path "/"
-			(page "1")
-		)
-	)
-	(embedded_fonts no)
 )

Commit message: pcb: finish psu upper
Parts:
- added C12: 3.3n, symbol Device:C
- added C13: 1u, symbol Device:C
- added C14, C17: 100n, symbol Device:C
- added C15, C16: 22u, symbol Device:C
- added C18: 10u, symbol Device:C
- added C19: 100u, symbol Device:C_US
- added L3: 1.5u, symbol Device:L
- added R7: 6.81k, symbol Device:R
- added R8: 22.1k, symbol Device:R
- added R9: 100k, symbol Device:R
Connections:
- net +1V0: now reaches U1.1 (VO)
- net +1V0: now also C15.1, C16.1, L3.2, R7.1
- net at U1.10 (SW1): now also U1.11 (SW2), C14.1, L3.1
- net at U1.12 (VBST): now also C14.2
- net POWER_IN: now reaches U1.13 (VIN)
- net POWER_IN: now also U1.14 (VCC), U1.7 (EN), C17.1, C18.1, C19.1
- net GND: now reaches U1.15 (EPAD)
- net GND: now also U1.5 (GND), U1.8 (PGND1), U1.9 (PGND2), C12.2, C13.2, C15.2, C16.2, C17.2, C18.2, C19.2, R8.2
- net at U1.2 (VFB): now also R7.2, R8.1
- net at U1.3 (VREG5): now also C13.1, R9.2
- net at U1.4 (SS): now also C12.1
- net at U1.6 (PG): now also R9.1
Other:
- moved on the sheet: U1

Commit message: pcb: connect upper and lower
Connections:
- net upper_right: now reaches R9.1, U1.6 (PG)
Changed lines of the file:
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@@
+		)
+	)
+	(hierarchical_label "upper_right"
+		(shape bidirectional)
+		(at 173.99 110.49 0)
+		(effects
+			(font
+				(size 1.27 1.27)
+			)
+			(justify left)
+		)
+	)
+	(hierarchical_label "upper_left"
+		(shape bidirectional)
+		(at 64.77 109.22 0)
+		(effects
+			(font
+				(size 1.27 1.27)
+			)
+			(justify left)
 		)
 	)
