File: pcb/power_mux.kicad_sch (KiCad schematic)
At the start: 0 parts

Commit message: pcb: usbc power supply + mux
Parts:
- added U7: TPS2116DRL, Package_TO_SOT_SMD:SOT-583-8, symbol Power_Management:TPS2116DRL
Connections:
- new net GND: U7.1 (GND), U7.4 (PR1), U7.5 (MODE)
- new net POWER_IN: U7.2 (VOUT), U7.7 (VOUT)
