File: pcb/power_source.kicad_sch (KiCad schematic)
At the start: 5 parts, among them J7 USB_C_Receptacle_USB2.0_14P

Commit message: fixed psd footprintgs and some routing
Changed lines of the file:
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@@
 		)
 	)
-	(label "5V_IN"
+	(global_label "5V_IN"
+		(shape input)
 		(at 185.42 60.96 0)
+		(fields_autoplaced yes)
 		(effects
 			(font
 				(size 1.27 1.27)
 			)
-			(justify left bottom)
+			(justify left)
+		)
+		(property "Intersheetrefs" "${INTERSHEET_REFS}"
+			(at 193.6062 60.96 0)
+			(hide yes)
+			(show_name no)
+			(do_not_autoplace no)
+			(effects
+				(font
+					(size 1.27 1.27)
+				)
+				(justify left)
+			)
 		)
 	)
