File: pcb/Powersupply.kicad_sch (KiCad schematic)
At the start: 39 parts, among them J2 Conn_02x04_Odd_Even, U5 TPS54325PWP.d, U6 TPS54294PWP

Commit message: pcb: mcu, sd card, jtag layout
Connections:
- net +1V0: now also L2.1; no longer L2.2
- net at C41.1, U5.10 (SW1), U5.11 (SW2): now also L2.2; no longer L2.1
Other:
- moved on the sheet: L2
Changed lines of the file:
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@@
+	(wire
+		(pts
+			(xy 104.14 40.64) (xy 118.11 40.64)
+		)
+		(stroke
+			(width 0)
+			(type default)
+		)
+	)
 	(wire
 		(pts
@@
 		(pts
 			(xy 233.68 74.93) (xy 233.68 77.47)
-		)
-		(stroke
-			(width 0)
-			(type default)
-		)
-	)
-	(wire
-		(pts
-			(xy 104.14 40.64) (xy 118.11 40.64)
 		)
 		(stroke
@@
 	(symbol
 		(lib_id "Device:L")
-		(at 195.58 33.02 90)
+		(at 195.58 33.02 270)
+		(mirror x)
 		(unit 1)
 		(body_style 1)
@@
 		(dnp no)
 		(property "Reference" "L2"
-			(at 192.786 34.544 90)
+			(at 198.374 34.544 90)
 			(show_name no)
 			(do_not_autoplace no)
@@
 		)
 		(property "Value" "1.5u"
-			(at 198.628 34.544 90)
+			(at 192.532 34.544 90)
 			(show_name no)
 			(do_not_autoplace no)
@@
 		)
 		(property "Extra" "lp>3.5A, lrms>3.1A"
-			(at 195.834 30.48 90)
-			(show_name no)
-			(do_not_autoplace no)
+			(at 195.326 30.48 90)
+			(show_name no)
+			(do_not_autoplace no)

Commit message: pcb: address feedback
- make rgb565 resistor ladder
- add 1v0 diode
- clean up pwr flags
- remove unused mcu-sd spi
- use labels in mcu
- fix broken rgb diode
- connect usblc pin 5 to vbus
Parts:
- added D3: red?, LED_SMD:LED_0805_2012Metric_Pad1.15x1.40mm_HandSolder, symbol Device:LED
- added R29: 1k, Resistor_SMD:R_0805_2012Metric_Pad1.20x1.40mm_HandSolder, symbol Device:R
- renumbered R29 to R30, R30 to R31, R31 to R32, R32 to R33, R33 to R34, R34 to R35, R35 to R36
Connections:
- net +1V0: now also R29.1
- net GND: now also D3.1 (K)
- net +3.3V renamed +3V3
- net +3.3VA renamed +3V3A
- new net: D3.2 (A), R29.2

Commit message: pcb
Parts:
- removed FB1: FerriteBead, Inductor_SMD:L_0805_2012Metric_Pad1.05x1.20mm_HandSolder, symbol Device:FerriteBead
- removed R36: 1, Resistor_SMD:R_0805_2012Metric_Pad1.20x1.40mm_HandSolder, symbol Device:R
- renumbered D1 to D4, D2 to D5, D3 to D6, J2 to J3, R25 to R31, R26 to R32, R27 to R33, R28 to R34, R29 to R35, R30 to R36, R31 to R37, R32 to R38, R33 to R39, R34 to R40, R35 to R41, U5 to U4, U6 to U5
