File: pcb/hello-world.kicad_sch (KiCad schematic)
At the start: 1 part, among them U2 TPS54325PWP

Commit message: pcb
Parts:
- removed U2: TPS54325PWP, PWP14_2P31X2P46, symbol TPS54325:TPS54325PWP
- added U1: TPS54325PWP.d, PWP14_2P31X2P46, symbol TPS54325:TPS54325PWP.d
Connections:
- new net: U1.14 (VCC), U1.5 (GND)
Other:
- removed sheet MCU
- removed sheet Powersupply
- removed sheet power_source
Changed lines of the file:
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@@
 	(generator_version "10.0")
 	(paper "A4")
+	(wire
+		(pts
+			(xy 119.38 91.44) (xy 107.95 91.44)
+		)
+		(stroke
+			(width 0)
+			(type default)
+		)
+	)
+	(wire
+		(pts
+			(xy 107.95 91.44) (xy 107.95 106.68)
+		)
+		(stroke
+			(width 0)
+			(type default)
+		)
+	)
+	(wire
+		(pts
+			(xy 107.95 106.68) (xy 119.38 106.68)
+		)
+		(stroke
+			(width 0)
+			(type default)
+		)
+	)
 	(symbol
-		(lib_id "TPS54325:TPS54325PWP")
-		(at 193.04 67.31 0)
+		(lib_id "TPS54325:TPS54325PWP.d")
+		(at 85.09 74.93 0)
 		(unit 1)
 		(body_style 1)
@@
 		(dnp no)
 		(fields_autoplaced yes)
-		(property "Reference" "U2"
-			(at 240.03 74.93 0)
+		(property "Reference" "U1"
+			(at 142.24 82.55 0)
 			(show_name no)
 			(do_not_autoplace no)
@@
 			)
 		)
-		(property "Value" "TPS54325PWP"
-			(at 240.03 77.47 0)
+		(property "Value" "TPS54325PWP.d"
+			(at 142.24 85.09 0)
 			(show_name no)
 			(do_not_autoplace no)
@@
 		)
 		(property "Footprint" "PWP14_2P31X2P46"
-			(at 207.01 85.09 0)
+			(at 93.98 119.38 0)
 			(hide yes)
 			(show_name no)
@@
 		)
 		(property "Datasheet" "https://www.ti.com/lit/gpn/tps54325"
-			(at 193.04 67.31 0)
+			(at 85.09 74.93 0)
 			(hide yes)
 			(show_name no)
@@
 		)
 		(property "Description" ""
-			(at 193.04 67.31 0)
+			(at 85.09 74.93 0)
 			(hide yes)
 			(show_name no)
@@
 			)
 		)
-		(pin "9"
+		(pin "1"
 		)
-		(pin "3"
-		)
-		(pin "5"
-		)
-		(pin "4"
-		)
-		(pin "14"
+		(pin "11"
 		)
 		(pin "10"
@@
 		(pin "15"
 		)
-		(pin "12"
+		(pin "13"
+		)
+		(pin "9"
+		)
+		(pin "3"
 		)
 		(pin "6"
 		)
-		(pin "13"
+		(pin "7"
+		)
+		(pin "4"
+		)
+		(pin "5"
+		)
+		(pin "12"
+		)
+		(pin "2"
+		)
+		(pin "14"
 		)
 		(pin "8"
 		)
-		(pin "1"
-		)
-		(pin "2"
-		)
-		(pin "11"
-		)
-		(pin "7"
-		)
 		(instances
 			(project "tdt4295"
-				(path "/603dd496-f9c4-4a31-9104-19eec41ebc98"
-					(reference "U2")
+				(path "/603dd496-f9c4-4a31-9104-19eec41ebc98/44fefbfa-6df6-4c0b-95cb-c8147218ca53"
+					(reference "U1")
 					(unit 1)
 				)
@@
 		)
 	)
-	(sheet
-		(at 54.61 38.1)
-		(size 31.75 12.7)
-		(exclude_from_sim no)
-		(in_bom yes)
-		(on_board yes)
-		(dnp no)
-		(fields_autoplaced yes)
-		(stroke
-			(width 0.1524)
-			(type solid)
-		)
-		(fill
-			(color 0 0 0 0)
-		)
-		(property "Sheetname" "power_source"
-			(at 54.61 37.3884 0)
-			(show_name no)
-			(do_not_autoplace no)
-			(effects
-				(font
-					(size 1.27 1.27)
-				)
-				(justify left bottom)
-			)
-		)
-		(property "Sheetfile" "power_source.kicad_sch"
-			(at 54.61 51.3846 0)
-			(show_name no)
-			(do_not_autoplace no)
-			(effects
-				(font
-					(size 1.27 1.27)
-				)
-				(justify left top)
-			)
-		)
-		(instances
-			(project "tdt4295"
-				(path "/603dd496-f9c4-4a31-9104-19eec41ebc98"
-					(page "7")
-				)
-			)
-		)
-	)
-	(sheet
-		(at 25.4 62.23)
-		(size 25.4 16.51)
-		(exclude_from_sim no)
-		(in_bom yes)
-		(on_board yes)
-		(dnp no)
-		(fields_autoplaced yes)
-		(stroke
-			(width 0.1524)
-			(type solid)
-		)
-		(fill
-			(color 0 0 0 0)
-		)
-		(property "Sheetname" "MCU"
-			(at 25.4 61.5184 0)
-			(show_name no)
-			(do_not_autoplace no)
-			(effects
-				(font
-					(size 1.27 1.27)
-				)
-				(justify left bottom)
-			)
-		)
-		(property "Sheetfile" "MCU.kicad_sch"
-			(at 25.4 79.3246 0)
-			(show_name no)
-			(do_not_autoplace no)
-			(effects
-				(font
-					(size 1.27 1.27)
-				)
-				(justify left top)
-			)
-		)
-		(instances
-			(project "tdt4295"
-				(path "/603dd496-f9c4-4a31-9104-19eec41ebc98"
-					(page "5")
-				)
-			)
-		)
-	)
-	(sheet
-		(at 25.4 38.1)
-		(size 25.4 12.7)
-		(exclude_from_sim no)
-		(in_bom yes)
-		(on_board yes)
-		(dnp no)
-		(fields_autoplaced yes)
-		(stroke
-			(width 0.1524)
-			(type solid)
-		)
-		(fill
-			(color 0 0 0 0)
-		)
-		(property "Sheetname" "Powersupply"
-			(at 25.4 37.3884 0)
-			(show_name no)
-			(do_not_autoplace no)
-			(effects
-				(font
-					(size 1.27 1.27)
-				)
-				(justify left bottom)
-			)
-		)
-		(property "Sheetfile" "Powersupply.kicad_sch"
-			(at 25.4 51.3846 0)
-			(show_name no)
-			(do_not_autoplace no)
-			(effects
-				(font
-					(size 1.27 1.27)
-				)
-				(justify left top)
-			)
-		)
-		(instances
-			(project "tdt4295"
-				(path "/603dd496-f9c4-4a31-9104-19eec41ebc98"
-					(page "4")
-				)
-			)
-		)
-	)
-	(sheet_instances
-		(path "/"
-			(page "1")
-		)
-	)
-	(embedded_fonts no)
 )
