File: pcb/_restore_backup_2026-09-10T09-00-11-938/STM32U535CE.kicad_sch (KiCad schematic)
At the start: 16 parts, among them J1 Conn_ST_STDC14, U6 STM32U535CETx, Y3 48MHz

Commit message: pcb: mcu schematic almost finished2
Connections:
- net at J1.12 (~{RST}): now also U6.7 (NRST)
Changed lines of the file:
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@@
+	(wire
+		(pts
+			(xy 76.2 45.72) (xy 76.2 102.87)
+		)
+		(stroke
+			(width 0)
+			(type default)
+		)
+	)
 	(wire
 		(pts
@@
 		)
 		(stroke
+			(width 0)
+			(type default)
+		)
+	)
+	(wire
+		(pts
+			(xy 76.2 102.87) (xy 72.39 102.87)
+		)
+		(stroke
+			(width 0)
+			(type default)
+		)
+	)
+	(wire
+		(pts
+			(xy 124.46 45.72) (xy 76.2 45.72)
+		)
+		(stroke
