File: pcb/_restore_backup_2026-09-15T12-27-13-418/MCU.kicad_sch (KiCad schematic)
At the start: 77 parts, among them J2 Conn_ST_STDC14, J6 Conn_ST_STDC14, J8 Micro_SD_Card, U10 STM32U595ZJTx, Y1 16MHz, Y5 16MHz

Commit message: add microsd
Parts:
- removed C67: 100nF, symbol Device:C
- removed C68: 1uF, symbol Device:C
- removed D10, D11, D12, D13, D2, D3, D4, D5, D6, D7, D8, D9: D_Zener_Filled, symbol Device:D_Zener_Filled
- removed J8: Micro_SD_Card, Connector_Card:microSD_HC_Molex_47219-2001, symbol Connector:Micro_SD_Card
- removed R33, R34, R39, R40, R41, R42: 22, symbol Device:R
- removed R43, R44, R45, R46, R47: 47k, symbol Device:R
Connections:
- net +3.3V: no longer C103.2, C104.2, C105.2, C106.2, C107.2, C108.2, C109.2, C110.2, C111.2, C112.2, C113.1, C114.1, C115.2, C116.2, C117.2, C118.2, C119.2, C120.2, C39.2, C40.2, C41.2, C42.2, C43.1, C44.1, C54.2, C55.2, C56.2, C57.2, C58.2, C59.2, C60.2, C61.2, C62.2, C63.2, C64.2, C83.2, J2.5 (GND), J2.7 (GND), J6.5 (GND), J6.7 (GND), STM32UF9NJH6Q_CUSTOM1.A1 (VSS), STM32UF9NJH6Q_CUSTOM1.A15 (VSS), STM32UF9NJH6Q_CUSTOM1.E10 (VSS), STM32UF9NJH6Q_CUSTOM1.F10 (VSS), STM32UF9NJH6Q_CUSTOM1.F6 (VSS), STM32UF9NJH6Q_CUSTOM1.F7 (VSS), STM32UF9NJH6Q_CUSTOM1.F9 (VSS), STM32UF9NJH6Q_CUSTOM1.G10 (VSS), STM32UF9NJH6Q_CUSTOM1.G6 (VSSDSI), STM32UF9NJH6Q_CUSTOM1.H10 (VSS), STM32UF9NJH6Q_CUSTOM1.H15 (VSS), STM32UF9NJH6Q_CUSTOM1.H2 (VSSDSI), STM32UF9NJH6Q_CUSTOM1.H6 (VSSDSI), STM32UF9NJH6Q_CUSTOM1.J10 (VSS), STM32UF9NJH6Q_CUSTOM1.J15 (VSS), STM32UF9NJH6Q_CUSTOM1.J2 (VSSDSI), STM32UF9NJH6Q_CUSTOM1.J6 (VSS), STM32UF9NJH6Q_CUSTOM1.K10 (VSS), STM32UF9NJH6Q_CUSTOM1.K6 (VSSA), STM32UF9NJH6Q_CUSTOM1.K7 (VSS), STM32UF9NJH6Q_CUSTOM1.K8 (VSS), STM32UF9NJH6Q_CUSTOM1.K9 (VSS), STM32UF9NJH6Q_CUSTOM1.L10 (VSS), STM32UF9NJH6Q_CUSTOM1.P12 (VSSSMPS), STM32UF9NJH6Q_CUSTOM1.R1 (VSS), STM32UF9NJH6Q_CUSTOM1.R15 (VSS), U10.107 (VSS), U10.120 (VSS), U10.130 (VSS), U10.143 (VSS), U10.16 (VSS), U10.30 (VSSA), U10.31 (VREF-), U10.38 (VSS), U10.51 (VSS), U10.61 (VSS), U10.71 (VSS), U10.83 (VSS), U10.94 (VSS), Y1.2 (G), Y1.4 (G), Y5.2 (G), Y5.4 (G)
- net CC1: no longer names the net of R38.1, U10.110 (PA15)
- net CC2: no longer names the net of U10.76 (PB15)
- net Drive_VBUS: no longer names the net of U10.40 (PA4)
- net fault_signal: no longer names the net of U10.41 (PA5)
- new net GND: C103.2, C104.2, C105.2, C106.2, C107.2, C108.2, C109.2, C110.2, C111.2, C112.2, C113.1, C114.1, C115.2, C116.2, C117.2, C118.2, C119.2, C120.2, C39.2, C40.2, C41.2, C42.2, C43.1, C44.1, C54.2, C55.2, C56.2, C57.2, C58.2, C59.2, C60.2, C61.2, C62.2, C63.2, C64.2, C83.2, J2.5 (GND), J2.7 (GND), J6.5 (GND), J6.7 (GND), STM32UF9NJH6Q_CUSTOM1.A1 (VSS), STM32UF9NJH6Q_CUSTOM1.A15 (VSS), STM32UF9NJH6Q_CUSTOM1.E10 (VSS), STM32UF9NJH6Q_CUSTOM1.F10 (VSS), STM32UF9NJH6Q_CUSTOM1.F6 (VSS), STM32UF9NJH6Q_CUSTOM1.F7 (VSS), STM32UF9NJH6Q_CUSTOM1.F9 (VSS), STM32UF9NJH6Q_CUSTOM1.G10 (VSS), STM32UF9NJH6Q_CUSTOM1.G6 (VSSDSI), STM32UF9NJH6Q_CUSTOM1.H10 (VSS), STM32UF9NJH6Q_CUSTOM1.H15 (VSS), STM32UF9NJH6Q_CUSTOM1.H2 (VSSDSI), STM32UF9NJH6Q_CUSTOM1.H6 (VSSDSI), STM32UF9NJH6Q_CUSTOM1.J10 (VSS), STM32UF9NJH6Q_CUSTOM1.J15 (VSS), STM32UF9NJH6Q_CUSTOM1.J2 (VSSDSI), STM32UF9NJH6Q_CUSTOM1.J6 (VSS), STM32UF9NJH6Q_CUSTOM1.K10 (VSS), STM32UF9NJH6Q_CUSTOM1.K6 (VSSA), STM32UF9NJH6Q_CUSTOM1.K7 (VSS), STM32UF9NJH6Q_CUSTOM1.K8 (VSS), STM32UF9NJH6Q_CUSTOM1.K9 (VSS), STM32UF9NJH6Q_CUSTOM1.L10 (VSS), STM32UF9NJH6Q_CUSTOM1.P12 (VSSSMPS), STM32UF9NJH6Q_CUSTOM1.R1 (VSS), STM32UF9NJH6Q_CUSTOM1.R15 (VSS), U10.107 (VSS), U10.120 (VSS), U10.130 (VSS), U10.143 (VSS), U10.16 (VSS), U10.30 (VSSA), U10.31 (VREF-), U10.38 (VSS), U10.51 (VSS), U10.61 (VSS), U10.71 (VSS), U10.83 (VSS), U10.94 (VSS), Y1.2 (G), Y1.4 (G), Y5.2 (G), Y5.4 (G)
Other:
- note removed: "ESD protection"
