File: pcb/_restore_backup_2026-09-15T12-27-13-418/Powersupply.kicad_sch (KiCad schematic)
At the start: 35 parts, among them J7 Conn_02x04_Odd_Even, U4 TPS54294PWP, U5 TPS54325PWP.d

Commit message: add microsd
Changed lines of the file:
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@@
 	)
 	(junction
-		(at 59.69 73.66)
-		(diameter 0)
-		(color 0 0 0 0)
-	)
-	(junction
 		(at 182.88 162.56)
 		(diameter 0)
@@
 	(wire
 		(pts
-			(xy 59.69 73.66) (xy 59.69 104.14)
-		)
-		(stroke
-			(width 0)
-			(type default)
-		)
-	)
-	(wire
-		(pts
 			(xy 168.91 40.64) (xy 151.13 40.64)
 		)
@@
 	(wire
 		(pts
-			(xy 45.72 73.66) (xy 59.69 73.66)
-		)
-		(stroke
-			(width 0)
-			(type default)
-		)
-	)
-	(wire
-		(pts
 			(xy 118.11 35.56) (xy 118.11 38.1)
 		)
@@
 	(wire
 		(pts
-			(xy 59.69 33.02) (xy 59.69 73.66)
+			(xy 59.69 33.02) (xy 59.69 104.14)
 		)
 		(stroke
@@
 			)
 		)
-		(property "Extra" "5V"
-			(at 52.07 36.576 0)
+		(property "Extra" "4.5V - 18V"
+			(at 55.118 36.83 0)
 			(show_name no)
 			(do_not_autoplace no)
@@
 					(unit 1)
 				)
-			)
-		)
-	)
-	(symbol
-		(lib_id "power:PWR_FLAG")
-		(at 45.72 73.66 0)
-		(unit 1)
-		(body_style 1)
-		(exclude_from_sim no)
-		(in_bom yes)
-		(on_board yes)
-		(in_pos_files yes)
-		(dnp no)
-		(fields_autoplaced yes)
-		(property "Reference" "#FLG01"
-			(at 45.72 71.755 0)
-			(hide yes)
-			(show_name no)
-			(do_not_autoplace no)
-			(effects
-				(font
-					(size 1.27 1.27)
-				)
-			)
-		)
-		(property "Value" "hub_pwr"
-			(at 45.72 68.58 0)
-			(show_name no)
-			(do_not_autoplace no)
-			(effects
-				(font
-					(size 1.27 1.27)
-				)
-			)
-		)
-		(property "Footprint" ""
-			(at 45.72 73.66 0)
-			(hide yes)
-			(show_name no)
-			(do_not_autoplace no)
-			(effects
-				(font
-					(size 1.27 1.27)
-				)
-			)
-		)
-		(property "Datasheet" ""
-			(at 45.72 73.66 0)
-			(hide yes)
-			(show_name no)
-			(do_not_autoplace no)
-			(effects
-				(font
-					(size 1.27 1.27)
-				)
-			)
-		)
-		(property "Description" "Special symbol for telling ERC where power comes from"
-			(at 45.72 73.66 0)
-			(hide yes)
-			(show_name no)
-			(do_not_autoplace no)
-			(effects
-				(font
-					(size 1.27 1.27)
-				)
-			)
-		)
-		(pin "1"
-		)
-		(instances
-			(project "tdt4295"
-				(path "/603dd496-f9c4-4a31-9104-19eec41ebc98/634870db-7705-458e-b29f-8b3e7772e7aa"
-					(reference "#FLG01")
-					(unit 1)
-				)
