File: pcb/_restore_backup_2026-09-15T12-27-13-418/usb_c.kicad_sch (KiCad schematic)
At the start: 8 parts, among them J3 USB_C_Receptacle_USB2.0_14P, U7 TPS2051CDBV, U8 USBLC6-2SC6

Commit message: add microsd
Parts:
- removed C65: 150uF, Package_TO_SOT_SMD:SOT-23-6, symbol Device:C_US
- removed C66: 0.1uF, symbol Device:C
- removed R32: 10k, symbol Device:R
Connections:
- net CC1 is gone; now on net GND: R31.2
- net CC2 is gone; now on net GND: R30.2
- net GND: no longer U7.2 (GND)
- net at J3.A4 (VBUS), J3.A9 (VBUS), J3.B4 (VBUS)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: no longer U7.1 (OUT)
- net Drive_VBUS: no longer names the net of U7.4 (EN)
- net POWER_IN: no longer names the net of U7.5 (IN)
- net fault_signal: no longer names the net of U7.3 (~{FLT})
