File: pcb/_restore_backup_2026-09-16T11-12-48-469/MCU.kicad_sch (KiCad schematic)
At the start: 54 parts, among them J6 Conn_ST_STDC14, J8 Micro_SD_Card, U10 STM32U595ZJTx, Y5 16MHz

Commit message: pcb: add VCP w/ESD protection
Parts:
- removed CR1: ESDALC6V1W5, SOT323-5L_STM, symbol ul_ESDALC6V1W5:ESDALC6V1W5
Connections:
- net at J6.13 (VCP_RX): no longer U10.102 (PA10)
- net at J6.14 (VCP_TX): no longer U10.101 (PA9)
- no-connect marks 2 -> 4
Other:
- moved on the sheet: C103, C104, C105, C106, C107, C108, C109, C110, C111, C112, C113, C114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
