File: pcb/_restore_backup_2026-09-17T15-35-30-941/MCU.kicad_sch (KiCad schematic)
At the start: 60 parts, among them J2 Conn_ST_STDC14, J3 Micro_SD_Card, SW1 SW_Push, SW2 SW_Push, U7 STM32U595ZJTx, Y2 16MHz

Commit message: added vddio pins and decoupling condensator
Parts:
- removed C74, C75, C76: 100nF, symbol Device:C
- removed R42: 100K, symbol Device:R
- removed SW2: SW_Push, Button_Switch_THT:SW_NKK_GW12LJP, symbol Switch:SW_Push
Connections:
- net +3.3V: no longer U7.131 (VDDIO2), U7.95 (VDDIO2)
- net USER_BUTTON: no longer names the net of U7.7 (PC13)
- no-connect marks 61 -> 64
Other:
- moved on the sheet: C50, C51, C52, C53, C54, C55, C56, C57, C58, C59
