File: pcb/_restore_backup_2026-09-17T17-20-11-015/Powersupply.kicad_sch (KiCad schematic)
At the start: 39 parts, among them J1 Conn_02x04_Odd_Even, U5 TPS54325PWP.d, U6 TPS54294PWP

Commit message: started removing errors from check
Connections:
- net POWER_IN is gone; now on net +1V0: C33.1, C34.1, C35.1, C36.1, C37.1, C44.1, C47.1, J1.1 (Pin_1), U5.13 (VIN), U5.14 (VCC), U5.7 (EN), U6.1 (VIN1), U6.16 (VIN2)
- net +1V0: now also C39.1, R13.2, R14.1, U5.2 (VFB), U5.4 (SS)
Changed lines of the file:
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@@
+	)
+	(junction
+		(at 118.11 43.18)
+		(diameter 0)
+		(color 0 0 0 0)
+	)
+	(junction
+		(at 134.62 60.96)
+		(diameter 0)
+		(color 0 0 0 0)
+	)
+	(junction
+		(at 99.06 45.72)
+		(diameter 0)
+		(color 0 0 0 0)
+	)
+	(junction
+		(at 186.69 33.02)
+		(diameter 0)
+		(color 0 0 0 0)
+	)
+	(junction
+		(at 205.74 60.96)
+		(diameter 0)
+		(color 0 0 0 0)
+	)
+	(junction
+		(at 130.81 162.56)
+		(diameter 0)
+		(color 0 0 0 0)
+	)
+	(junction
+		(at 233.68 74.93)
+		(diameter 0)
+		(color 0 0 0 0)
+	)
+	(junction
+		(at 38.1 162.56)
+		(diameter 0)
+		(color 0 0 0 0)
+	)
+	(junction
+		(at 59.69 33.02)
+		(diameter 0)
+		(color 0 0 0 0)
+	)
+	(junction
+		(at 158.75 60.96)
+		(diameter 0)
+		(color 0 0 0 0)
+	)
+	(junction
+		(at 50.8 162.56)
+		(diameter 0)
+		(color 0 0 0 0)
+	)
+	(junction
+		(at 20.32 125.73)
+		(diameter 0)
+		(color 0 0 0 0)
+	)
+	(junction
+		(at 87.63 60.96)
+		(diameter 0)
+		(color 0 0 0 0)
+	)
+	(junction
+		(at 248.92 144.78)
+		(diameter 0)
+		(color 0 0 0 0)
+	)
+	(junction
+		(at 78.74 162.56)
+		(diameter 0)
+		(color 0 0 0 0)
+	)
+	(junction
+		(at 203.2 104.14)
+		(diameter 0)
+		(color 0 0 0 0)
+	)
+	(junction
+		(at 105.41 133.35)
+		(diameter 0)
+		(color 0 0 0 0)
+	)
+	(junction
+		(at 248.92 127)
+		(diameter 0)
+		(color 0 0 0 0)
+	)
+	(junction
+		(at 228.6 127)
+		(diameter 0)
+		(color 0 0 0 0)
+	)
+	(junction
+		(at 171.45 104.14)
+		(diameter 0)
+		(color 0 0 0 0)
+	)
+	(junction
+		(at 118.11 38.1)
+		(diameter 0)
+		(color 0 0 0 0)
+	)
+	(junction
+		(at 130.81 135.89)
+		(diameter 0)
+		(color 0 0 0 0)
+	)
+	(junction
+		(at 118.11 33.02)
+		(diameter 0)
+		(color 0 0 0 0)
+	)
+	(junction
+		(at 176.53 162.56)
+		(diameter 0)
+		(color 0 0 0 0)
+	)
+	(junction
+		(at 107.95 60.96)
+		(diameter 0)
+		(color 0 0 0 0)
 	)
 	(junction
@@
 	)
 	(junction
-		(at 134.62 60.96)
-		(diameter 0)
-		(color 0 0 0 0)
-	)
-	(junction
-		(at 99.06 45.72)
-		(diameter 0)
-		(color 0 0 0 0)
-	)
-	(junction
-		(at 186.69 33.02)
-		(diameter 0)
-		(color 0 0 0 0)
-	)
-	(junction
-		(at 205.74 60.96)
-		(diameter 0)
-		(color 0 0 0 0)
-	)
-	(junction
-		(at 130.81 162.56)
-		(diameter 0)
-		(color 0 0 0 0)
-	)
-	(junction
-		(at 233.68 74.93)
-		(diameter 0)
-		(color 0 0 0 0)
-	)
-	(junction
-		(at 38.1 162.56)
-		(diameter 0)
-		(color 0 0 0 0)
-	)
-	(junction
-		(at 59.69 33.02)
-		(diameter 0)
-		(color 0 0 0 0)
-	)
-	(junction
-		(at 158.75 60.96)
-		(diameter 0)
-		(color 0 0 0 0)
-	)
-	(junction
-		(at 50.8 162.56)
-		(diameter 0)
-		(color 0 0 0 0)
-	)
-	(junction
-		(at 20.32 125.73)
-		(diameter 0)
-		(color 0 0 0 0)
-	)
-	(junction
-		(at 87.63 60.96)
-		(diameter 0)
-		(color 0 0 0 0)
-	)
-	(junction
-		(at 248.92 144.78)
-		(diameter 0)
-		(color 0 0 0 0)
-	)
-	(junction
-		(at 78.74 162.56)
-		(diameter 0)
-		(color 0 0 0 0)
-	)
-	(junction
-		(at 203.2 104.14)
-		(diameter 0)
-		(color 0 0 0 0)
-	)
-	(junction
-		(at 105.41 133.35)
-		(diameter 0)
-		(color 0 0 0 0)
-	)
-	(junction
-		(at 248.92 127)
-		(diameter 0)
-		(color 0 0 0 0)
-	)
-	(junction
-		(at 228.6 127)
-		(diameter 0)
-		(color 0 0 0 0)
-	)
-	(junction
-		(at 171.45 104.14)
-		(diameter 0)
-		(color 0 0 0 0)
-	)
-	(junction
-		(at 130.81 135.89)
-		(diameter 0)
-		(color 0 0 0 0)
-	)
-	(junction
-		(at 118.11 33.02)
-		(diameter 0)
-		(color 0 0 0 0)
-	)
-	(junction
-		(at 176.53 162.56)
-		(diameter 0)
-		(color 0 0 0 0)
-	)
-	(junction
-		(at 107.95 60.96)
+		(at 240.03 127)
+		(diameter 0)
+		(color 0 0 0 0)
+	)
+	(junction
+		(at 148.59 162.56)
+		(diameter 0)
+		(color 0 0 0 0)
+	)
+	(junction
+		(at 118.11 60.96)
+		(diameter 0)
+		(color 0 0 0 0)
+	)
+	(junction
+		(at 99.06 60.96)
+		(diameter 0)
+		(color 0 0 0 0)
+	)
+	(junction
+		(at 151.13 60.96)
 		(diameter 0)
 		(color 0 0 0 0)
@@
 	)
 	(junction
-		(at 240.03 127)
-		(diameter 0)
-		(color 0 0 0 0)
-	)
-	(junction
-		(at 148.59 162.56)
-		(diameter 0)
-		(color 0 0 0 0)
-	)
-	(junction
-		(at 118.11 60.96)
-		(diameter 0)
-		(color 0 0 0 0)
-	)
-	(junction
-		(at 99.06 60.96)
-		(diameter 0)
-		(color 0 0 0 0)
-	)
-	(junction
-		(at 151.13 60.96)
-		(diameter 0)
-		(color 0 0 0 0)
-	)
-	(junction
 		(at 251.46 127)
 		(diameter 0)
@@
 	(junction
 		(at 233.68 77.47)
+		(diameter 0)
+		(color 0 0 0 0)
+	)
+	(junction
+		(at 118.11 40.64)
 		(diameter 0)
 		(color 0 0 0 0)
@@
 	(wire
 		(pts
+			(xy 99.06 38.1) (xy 118.11 38.1)
+		)
+		(stroke
+			(width 0)
+			(type default)
+		)
+	)
+	(wire
+		(pts
 			(xy 158.75 55.88) (xy 158.75 60.96)
 		)
@@
 	(wire
 		(pts
-			(xy 116.84 35.56) (xy 116.84 45.72)
-		)
-		(stroke
-			(width 0)
-			(type default)
-		)
-	)
-	(wire
-		(pts
 			(xy 130.81 162.56) (xy 148.59 162.56)
 		)
@@
 	(wire
 		(pts
+			(xy 118.11 43.18) (xy 118.11 45.72)
+		)
+		(stroke
+			(width 0)
+			(type default)
+		)
+	)
+	(wire
+		(pts
 			(xy 240.03 127) (xy 248.92 127)
 		)
@@
 	(wire
 		(pts
+			(xy 118.11 35.56) (xy 118.11 38.1)
+		)
+		(stroke
+			(width 0)
+			(type default)
+		)
+	)
+	(wire
+		(pts
 			(xy 78.74 104.14) (xy 91.44 104.14)
 		)
@@
 	(wire
 		(pts
+			(xy 118.11 40.64) (xy 118.11 43.18)
+		)
+		(stroke
+			(width 0)
+			(type default)
+		)
+	)
+	(wire
+		(pts
 			(xy 59.69 104.14) (xy 78.74 104.14)
 		)
@@
 	(wire
 		(pts
-			(xy 118.11 35.56) (xy 116.84 35.56)
-		)
-		(stroke
-			(width 0)
-			(type default)
-		)
-	)
-	(wire
-		(pts
 			(xy 212.09 24.13) (xy 212.09 33.02)
 		)
@@
 	(wire
 		(pts
+			(xy 118.11 38.1) (xy 118.11 40.64)
+		)
+		(stroke
+			(width 0)
+			(type default)
+		)
+	)
+	(wire
+		(pts
 			(xy 127 153.67) (xy 177.8 153.67)
 		)
@@
 	(wire
 		(pts
-			(xy 99.06 38.1) (xy 118.11 38.1)
-		)
-		(stroke
-			(width 0)
-			(type default)
-		)
-	)
-	(wire
-		(pts
 			(xy 251.46 127) (xy 255.27 127)
 		)
@@
 		)
 		(stroke
-			(width 0)
-			(type default)
-		)
-	)
-	(wire
-		(pts
-			(xy 116.84 45.72) (xy 118.11 45.72)
-		)
-		(stroke
