File: pcb/_restore_backup_2026-09-17T17-20-11-015/fpga.kicad_sch (KiCad schematic)
At the start: 45 parts, among them U1 XC7A50T-FTG256, U2 410-251-B, U3 S70KL1283GABHI020, U4 W25Q128JVS, Y1 ASE-20MHz

Commit message: started removing errors from check
Changed lines of the file:
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@@
 	(wire
 		(pts
-			(xy 111.76 87.63) (xy 110.49 87.63)
-		)
-		(stroke
-			(width 0)
-			(type default)
-		)
-	)
-	(wire
-		(pts
 			(xy 157.48 66.04) (xy 157.48 67.31)
 		)
@@
 	(symbol
 		(lib_id "power:+3V3")
-		(at 111.76 87.63 270)
+		(at 110.49 87.63 270)
 		(unit 1)
 		(body_style 1)
@@
 		(dnp no)
 		(property "Reference" "#PWR04"
-			(at 107.95 87.63 0)
+			(at 106.68 87.63 0)
 			(hide yes)
 			(show_name no)
@@
 		)
 		(property "Value" "+3V3"
-			(at 116.078 87.63 90)
+			(at 114.808 87.63 90)
 			(show_name no)
 			(do_not_autoplace no)
@@
 		)
 		(property "Footprint" ""
-			(at 111.76 87.63 0)
+			(at 110.49 87.63 0)
 			(hide yes)
 			(show_name no)
@@
 		)
 		(property "Datasheet" ""
-			(at 111.76 87.63 0)
+			(at 110.49 87.63 0)
 			(hide yes)
 			(show_name no)
@@
 		)
 		(property "Description" "Power symbol creates a global label with name \"+3V3\""
-			(at 111.76 87.63 0)
+			(at 110.49 87.63 0)
 			(hide yes)
 			(show_name no)
